Commit message: 20251203_lidar6

File: src/rosmaster_description/urdf/ugv.urdf.xacro (robot description, xacro)
@@ -190,6 +190,6 @@
     <parent link="base_link"/>
     <child link="laser_link"/>
-    <!-- LIDAR를 전면을 바라보도록 yaw 회전을 0으로 설정 -->
-    <origin xyz="${LIDAR_X} 0 ${LIDAR_Z}" rpy="0 0 0"/>
+    <!-- LIDAR 데이터가 실제 전면과 일치하도록 180도 회전 -->
+    <origin xyz="${LIDAR_X} 0 ${LIDAR_Z}" rpy="0 0 ${PI}"/>
   </joint>
   <joint name="imu_joint" type="fixed">
